Commit message: converison

File: mujoco_models/sawyer/sawyer.urdf (robot description, URDF)
Before this commit: robot sawyer, 21 links, 20 joints
Links:
- link head: geometry collision sphere radius=0.18; visual mesh filename=sawyer_pv/head.stl
- link pedestal: geometry collision cylinder length=0.62 radius=0.18; visual mesh filename=sawyer_pv/pedestal.stl
- link right_arm_base_link: geometry collision cylinder length=0.24 radius=0.08; visual mesh filename=sawyer_pv/base.stl
- link right_l0: geometry collision sphere radius=0.07; visual mesh filename=sawyer_mp3/l0.stl
- link right_l1: geometry collision sphere radius=0.07; visual mesh filename=sawyer_mp3/l1.stl
- link right_l2: geometry collision cylinder length=0.35 radius=0.06; visual mesh filename=sawyer_pv/l2.stl
- link right_l3: geometry collision sphere radius=0.06; visual mesh filename=sawyer_pv/l3.stl
- link right_l4: geometry collision cylinder length=0.36 radius=0.045; visual mesh filename=sawyer_pv/l4.stl
- link right_l5: geometry collision sphere radius=0.06; visual mesh filename=sawyer_pv/l5.stl
- link right_l6: geometry collision cylinder length=0.05 radius=0.065; visual mesh filename=sawyer_mp1/l6.stl

Commit message: file renaming and restructuring

File: mujoco_models/sawyer/sawyer.urdf (robot description, URDF)
Before this commit: robot sawyer, 21 links, 20 joints
Links:
- added link right_l1_2, mass 1.0E-08; collision cylinder length=0.14 radius=0.07
- added link right_l2_2, mass 1.0E-08; collision sphere radius=0.06
- added link right_l4_2, mass 1.0E-08; collision sphere radius=0.06
- link head: geometry collision sphere radius=0.18; visual mesh filename=package://head.stl scale=1 1 1
- link pedestal: geometry collision cylinder length=0.62 radius=0.18; visual mesh filename=package://pedestal.stl scale=1 1 1
- link right_arm_base_link: geometry collision cylinder length=0.24 radius=0.08; visual mesh filename=package://base.stl scale=1 1 1
- link right_hand: geometry collision cylinder length=0.03 radius=0.035
- link right_l0: geometry collision sphere radius=0.07; visual mesh filename=package://l0.stl scale=1 1 1
- link right_l1: geometry collision sphere radius=0.07; visual mesh filename=package://l1.stl scale=1 1 1
- link right_l2: mass 1.7251 -> 1.745; geometry collision cylinder length=0.34 radius=0.06; visual mesh filename=package://l2.stl scale=1 1 1
- link right_l3: mass 2.4743 -> 2.5097; geometry collision sphere radius=0.06; visual mesh filename=package://l3.stl scale=1 1 1
- link right_l4: mass 1.0433 -> 1.1136; geometry collision cylinder length=0.30 radius=0.045; visual mesh filename=package://l4.stl scale=1 1 1
- link right_l5: mass 1.5343 -> 1.5625; geometry collision sphere radius=0.06; visual mesh filename=package://l5.stl scale=1 1 1
- link right_l6: geometry collision cylinder length=0.05 radius=0.055; visual mesh filename=package://l6.stl scale=1 1 1
Joints:
- added joint right_j1_2: type fixed, parent right_l1, child right_l1_2, origin xyz=0 0 0 rpy=0 0 0, axis 0 0 1
- added joint right_j2_2: type fixed, parent right_l2, child right_l2_2, origin xyz=0 0 0 rpy=0 0 0, axis 0 0 1
- added joint right_j4_2: type fixed, parent right_l4, child right_l4_2, origin xyz=0 0 0 rpy=0 0 0, axis 0 0 1
- joint head_pan: limit lower=-5.1477 upper=0.9559 effort=8 velocity=1.8 -> lower=-5.0952 upper=0.9064 effort=8 velocity=1.8
- joint right_j1: limit lower=-3.8183 upper=2.2824 effort=80.0 velocity=1.328 -> lower=-3.8095 upper=2.2736 effort=80.0 velocity=1.328
- joint right_j2: limit lower=-3.0514 upper=3.0514 effort=40.0 velocity=1.957 -> lower=-3.0426 upper=3.0426 effort=40.0 velocity=1.957
- joint right_j3: limit lower=-3.0514 upper=3.0514 effort=40.0 velocity=1.957 -> lower=-3.0439 upper=3.0439 effort=40.0 velocity=1.957
- joint right_j4: limit lower=-2.9842 upper=2.9842 effort=9.0 velocity=3.485 -> lower=-2.9761 upper=2.9761 effort=9.0 velocity=3.485
- joint right_j5: limit lower=-2.9842 upper=2.9842 effort=9.0 velocity=3.485 -> lower=-2.9761 upper=2.9761 effort=9.0 velocity=3.485
- joint right_j6: limit lower=-4.7104 upper=4.7104 effort=9.0 velocity=4.545 -> lower=-4.7124 upper=4.7124 effort=9.0 velocity=4.545

Commit message: added environment models

File: mujoco_models/sawyer/sawyer.urdf (robot description, URDF)
Before this commit: robot sawyer, 24 links, 23 joints
Links:
- link torso: geometry visual box size=0.1 0.1 0.1
